File: Design/Design.kicad_sch (KiCad schematic)
At the start: 0 parts

Commit message: started schematic
Parts:
- added J1: ~, symbol my_lib:J1
- added J2: ~, symbol my_lib:J2
- added J3: FTDI, symbol my_lib:J3
- added U1: ATMEGA328P-A, symbol my_lib:ATMEGA328P-A
Connections:
- new net test: U1.11 (PD7)
